File: Rpi-CAN.brd (EAGLE design)
At the start: 35.6 x 43.8 mm, 22 parts, among them IC1 SN65HVD233-HT, IC2 MCP2510SO, IC3 XC6221B332MR, Q1 20M

Commit message: Added resitor for connecting Raspberry Pi 5V rail to CAN optional power.
Parts:
- added R7: 0R, rcl:R0805
Connections:
- new net N$5: R7.2, X3.9
- net +5V: now also R7.1
Routing:
- net N$5: track 0.00 -> 26.0 mm, vias 0 -> 1
- net +5V: track 17.8 -> 22.8 mm
Changed lines of the file:
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@@
 <layer number="21" name="tPlace" color="7" fill="1" visible="yes" active="yes"/>
 <layer number="22" name="bPlace" color="7" fill="1" visible="yes" active="yes"/>
-<layer number="23" name="tOrigins" color="15" fill="1" visible="no" active="yes"/>
-<layer number="24" name="bOrigins" color="15" fill="1" visible="no" active="yes"/>
+<layer number="23" name="tOrigins" color="15" fill="1" visible="yes" active="yes"/>
+<layer number="24" name="bOrigins" color="15" fill="1" visible="yes" active="yes"/>
 <layer number="25" name="tNames" color="7" fill="1" visible="yes" active="yes"/>
 <layer number="26" name="bNames" color="7" fill="1" visible="yes" active="yes"/>
@@
 <attribute name="VALUE" x="28.575" y="20.32" size="1.27" layer="27" rot="R90"/>
 </element>
+<element name="R7" library="rcl" package="R0805" value="0R" x="26.035" y="13.97" rot="R90"/>
 </elements>
 <signals>
@@
 <wire x1="30.45" y1="14.92" x2="29.525" y2="14.92" width="0.3048" layer="1"/>
 <wire x1="29.525" y1="14.92" x2="29.21" y2="14.605" width="0.3048" layer="1"/>
+<contactref element="R7" pad="1"/>
+<wire x1="26.035" y1="13.02" x2="26.035" y2="12.7" width="0.3048" layer="1"/>
+<wire x1="26.035" y1="12.7" x2="26.67" y2="12.065" width="0.3048" layer="1"/>
+<wire x1="26.67" y1="12.065" x2="30.48" y2="12.065" width="0.3048" layer="1"/>
 </signal>
 <signal name="N$1">
@@
 <via x="27.305" y="16.51" extent="1-16" drill="0.3048"/>
 <via x="23.495" y="12.7" extent="1-16" drill="0.3048"/>
-<via x="27.305" y="12.7" extent="1-16" drill="0.3048"/>
+<via x="27.94" y="13.335" extent="1-16" drill="0.3048"/>
 <via x="34.925" y="16.51" extent="1-16" drill="0.3048"/>
 <via x="34.925" y="19.685" extent="1-16" drill="0.3048"/>
@@
 <wire x1="26.035" y1="22.86" x2="26.035" y2="21.905" width="0.3048" layer="1"/>
 </signal>
+<signal name="N$5">
+<contactref element="X3" pad="9"/>
+<contactref element="R7" pad="2"/>
+<wire x1="26.035" y1="14.92" x2="26.035" y2="15.875" width="0.3048" layer="1"/>
+<wire x1="26.035" y1="15.875" x2="22.86" y2="19.05" width="0.3048" layer="16"/>
+<wire x1="22.86" y1="19.05" x2="22.86" y2="27.94" width="0.3048" layer="16"/>
+<wire x1="22.86" y1="27.94" x2="25.7048" y2="30.7848" width="0.3048" layer="16"/>
+<wire x1="33.3248" y1="30.7848" x2="25.7048" y2="30.7848" width="0.3048" layer="16"/>
+<via x="26.035" y="15.875" extent="1-16" drill="0.3048"/>
+</signal>
 </signals>
